File: PowerAmp.kicad_sch (KiCad schematic)
At the start: 0 parts

Commit message: Power Amp Schematic
Parts:
- added C1, C2, C3, C4: 4700pF 250V, symbol Device:C
- added C10, C9: 330pF 500V, symbol Device:C
- added C11, C12: 6800pF 100V, symbol Device:C
- added C13, C14, C15, C16: 330uF 100V, symbol Device:C_Polarized
- added C17, C18, C6, C7: 0.1uF 250V, symbol Device:C
- added C19, C20: 3300uF 50V, symbol Device:C_Polarized
- added C21, C22: 22uF 200V, symbol Device:C_Polarized
- added C23, C24: 100uF 25V, symbol Device:C_Polarized
- added C26: 10uF 16V, symbol Device:C
- added C28: 10uF 25V, symbol Device:C_Polarized
- added C29: 1500pF 50V, symbol Device:C
- added C30, C31: 330pF 50V, symbol Device:C
- added C32, C33: 0.022uF 250V, symbol Device:C
- added D1, D2: HZ6A1L, symbol Device:D_Zener
- added D10, D11, D12, D9: MA165, Diode_THT:D_DO-35_SOD27_P7.62mm_Horizontal, symbol Diode:1N4448
- added D13, D14: 1SR139-400, Diode_THT:D_DO-35_SOD27_P7.62mm_Horizontal, symbol Diode:1N4448
- added D15: LN1VB60, Diode_THT:Diode_Bridge_Vishay_GBU, symbol Diode_Bridge:GBU4A
- added D16, D17: HZ9A2L, symbol Device:D_Zener
- added D18, D19, D20, D21: HZ153L, symbol Device:D_Zener
- added D3, D4: MA167, Diode_THT:D_DO-35_SOD27_P7.62mm_Horizontal, symbol Diode:1N4448
- added D5, D6: 1SS83, Diode_THT:D_DO-35_SOD27_P7.62mm_Horizontal, symbol Diode:1N4448
- added D7, D8: 1Z15A, symbol Device:D_Zener
- added IC1, IC2: NJM4580D-D, DIP8_NWJ, symbol 2026-06-02_03-55-29:NJM4580D
- added K1, K2: Conn_01x02_Pin, symbol Connector:Conn_01x02_Pin
- added K3: Conn_01x04_Pin, symbol Connector:Conn_01x04_Pin
- added K4: Conn_01x03_Pin, symbol Connector:Conn_01x03_Pin
- added Q1, Q2, Q26, Q7, Q8: 2SA1376-K/U, Package_TO_SOT_THT:TO-92_Inline, symbol Transistor_BJT:2SA1015
- added Q10, Q13, Q14, Q9: 2SA1145-Y, Package_TO_SOT_THT:TO-92_Inline, symbol Transistor_BJT:2SA1015
- added Q11, Q12, Q15, Q16: 2SC2705-Y, Package_TO_SOT_THT:TO-92_Inline, symbol Transistor_BJT:2SC1815
- added Q17: 2SA1507-S/T, Package_TO_SOT_THT:TO-92_Inline, symbol Transistor_BJT:2SA1015
- added Q18, Q25: 2SC3902-S/T, Package_TO_SOT_THT:TO-92_Inline, symbol Transistor_BJT:2SC1815
- added Q19: 2SC4793, Package_TO_SOT_THT:TO-92_Inline, symbol Transistor_BJT:2SC1815
- added Q20: 2SA1837, Package_TO_SOT_THT:TO-92_Inline, symbol Transistor_BJT:2SA1015
- added Q21, Q23: 2SC5949-O, Package_TO_SOT_THT:TO-92_Inline, symbol Transistor_BJT:2SC1815
- added Q22, Q24: 2SA2121-O, Package_TO_SOT_THT:TO-92_Inline, symbol Transistor_BJT:2SA1015
- added Q27, Q3, Q4, Q5, Q6: 2SC3478-K/U, Package_TO_SOT_THT:TO-92_Inline, symbol Transistor_BJT:2SC1815
- added R1: 470 1/6W, symbol Device:R
- added R10, R11, R12, R17, R18, R19, R20, R9: 22 1/6W, symbol Device:R
- added R13, R14, R15, R16: 2.4k 1/6W, symbol Device:R
- added R2: 24k 1/4W, symbol Device:R
- added R21, R22, R23, R24: 5.6k 1/6W, symbol Device:R
- added R25, R26, R27, R28, R33, R68, R69: 1k 1/4W, symbol Device:R
- added R29, R30, R31, R32: 150 1/4W, symbol Device:Fuse
- added R3, R4: 100 1/6W, symbol Device:R
- added R34: 240 1/4W, symbol Device:R
- added R35: 75k 1/4W, symbol Device:R
- added R36: 47 2W, symbol Device:R
- added R37, R38, R66, R67: 100 2W, symbol Device:R
- added R39, R40: 2.2 1/4W, symbol Device:R
- added R41, R42: 680 1/4W, symbol Device:R
- added R43, R44: 390 1/4W, symbol Device:R
- added R45, R46, R49, R50: 0.22 2W, symbol Device:R
- added R5, R6, R7, R8: 15k 1/6W, symbol Device:R
- added R51, R52: 330 1/6W, symbol Device:R
- added R53, R54: 5.6k 3W, symbol Device:R
- added R55, R56: 4.42k 1/2W, symbol Device:R
- added R57, R58: 33k 1/6W, symbol Device:R
- added R59, R60: 0.47 1/4W, symbol Device:Fuse
- added R61: 2.21k 2W, symbol Device:R
- added R62, R64: 332 1/4W, symbol Device:R
- added R63: 270k 1/6W, symbol Device:R
- added R70: 715 1/4W, symbol Device:R
- added R71, R72: 3.9k 3W, symbol Device:R
- added TP1: 10 mV Test Point 1, symbol Connector:Conn_01x02_Pin
- added TPA_1V2, TPB_1V2: +1.2V, symbol Connector:Conn_01x01_Pin
- added VR1: 200, symbol Device:R_Potentiometer_US
Connections:
- new net: Q21.1 (E), R41.1, R45.1, R51.1
- new net: Q10.1 (E), Q14.3 (B), R26.1
- new net: D12.2 (A), R16.1
- new net: C4.1, D21.1 (K), Q12.3 (B), Q8.2 (C), R16.2
- new net: Q16.1 (E), R32.1
- new net: Q11.2 (C), Q12.2 (C), Q15.2 (C), Q16.2 (C), Q18.1 (E)
- new net: Q12.1 (E), Q16.3 (B), R28.2
- new net: C23.1, D7.1 (K), IC1.8 (V+), IC2.8 (V+), R5.1, R53.2, R6.1, R71.2
- new net: Q24.1 (E), R50.2
- new net: Q22.3 (B), Q24.3 (B), R40.1
- new net: K4.3 (Pin_3), R66.1
- new net: C11.1, Q27.3 (B), R41.2, R43.2
- new net: R34.1, VR1.3
- new net: Q25.3 (B), R33.1, R34.2
- new net: C28.2, C29.1, IC2.3 (A+INPUT), R2.1
- new net: Q13.1 (E), R29.2
- new net: C10.1, D4.1 (K), D6.1 (K), Q18.2 (C), Q20.3 (B), Q25.1 (E), TPB_1V2.1 (Pin_1), VR1.1, VR1.2
- new net: C12.1, D4.2 (A), Q26.2 (C)
- new net: Q7.1 (E), R19.1
- new net: R17.1, R18.1, R19.2, R20.2, R55.1, R56.1, R62.2
- new net: C31.2, IC2.7 (B_OUTPUT), R62.1, R69.2
- new net: Q19.1 (E), R36.2, R39.1
- new net: Q21.3 (B), Q23.3 (B), R39.2
- new net: C30.2, IC2.1 (A_OUTPUT), R64.1, R68.2
- new net: C30.1, IC2.2 (A-INPUT), R68.1, R70.1
- new net: C24.2, D8.2 (A), IC1.4 (V-), IC2.4 (V-), R54.2, R7.1, R72.2, R8.1
- new net: C31.1, IC2.6 (B-INPUT), R69.1, R70.2
- new net: C2.2, D19.2 (A), Q10.3 (B), Q6.2 (C), R14.1
- new net: D10.1 (K), R14.2
- new net: Q20.2 (C), R36.1, R40.2
- new net: R3.1, R4.1, R61.2, R64.2
- new net: Q2.3 (B), Q4.3 (B), R4.2
- new net: Q8.1 (E), R20.1
- new net: Q8.3 (B), R12.1, R8.2
- new net: Q5.1 (E), R17.2
- new net: C4.2, R24.2
- new net: Q11.1 (E), Q15.3 (B), R27.2
- new net: Q15.1 (E), R31.1
- new net: Q10.2 (C), Q13.2 (C), Q14.2 (C), Q17.1 (E), Q9.2 (C)
- new net: C26.2, IC1.7 (B_OUTPUT), R61.1
- new net: Q22.1 (E), R42.2, R46.2, R52.1
- new net: Q23.1 (E), R49.1
- new net: C2.1, R22.1
- new net: D11.2 (A), R15.1
- new net: D16.1 (K), D17.1 (K)
- new net: C26.1, D16.2 (A), IC1.6 (B-INPUT), R58.1
- new net: Q13.3 (B), Q9.1 (E), R25.1
- new net: C1.2, D18.2 (A), Q5.2 (C), Q9.3 (B), R13.1
- new net: D9.1 (K), R13.2
- new net: K4.1 (Pin_1), R67.1
- new net: R52.2, TP1.1 (Pin_1)
- new net: R51.2, TP1.2 (Pin_2)
- new net: Q17.2 (C), Q25.2 (C), R33.2
- new net: D1.2 (A), Q17.3 (B), R35.2
- new net: D15.2, R59.1
- new net: D15.3, R60.1
- new net: Q2.1 (E), R10.1
- new net: Q6.3 (B), R10.2, R6.2
- new net: C11.2, D3.1 (K), Q27.2 (C)
- new net: Q14.1 (E), R30.2
- new net: Q4.1 (E), R12.2
- new net: D2.1 (K), Q18.3 (B), R35.1
- new net: C9.1, D3.2 (A), D5.2 (A), Q19.3 (B), TPA_1V2.1 (Pin_1)
- new net: Q5.3 (B), R5.2, R9.2
- new net: C3.2, R23.2
- new net: Q1.1 (E), R9.1
- new net: Q1.3 (B), Q3.3 (B), R3.2
- new net: Q6.1 (E), R18.2
- new net: C3.1, D20.1 (K), Q11.3 (B), Q7.2 (C), R15.2
- new net: Q7.3 (B), R11.1, R7.2
- new net: Q3.1 (E), R11.2
- new net: C12.2, Q26.3 (B), R42.1, R44.1
- new net: C28.1, R1.2, R63.2
- new net: C1.1, R21.1
- new net: IC1.5 (B+INPUT), R57.1
- new net +66V: C19.2, C21.1, C32.1, D13.2 (A), D5.1 (K), K3.2 (Pin_2), Q21.2 (C), Q23.2 (C), R53.1, R71.1
- new net +74.8V: C13.1, C15.1, C7.1, D1.1 (K), D10.2 (A), D18.1 (K), D19.1 (K), D9.2 (A), Q3.2 (C), Q4.2 (C), R21.2, R22.2, R25.2, R26.2, R29.1, R30.1, R37.2, R66.2
- new net +78.9V: C17.1, C19.1, D13.1 (K), D15.1 (+), Q19.2 (C), R37.1
- new net -66V: C20.1, C22.2, C32.2, D14.1 (K), D6.2 (A), K3.4 (Pin_4), Q22.2 (C), Q24.2 (C), R54.1, R72.1
- new net -74.8V: C14.2, C16.2, C6.1, D11.1 (K), D12.1 (K), D2.2 (A), D20.2 (A), D21.2 (A), Q1.2 (C), Q2.2 (C), R23.1, R24.1, R27.1, R28.1, R31.2, R32.2, R38.1, R67.2
- new net -78.9V: C18.2, C20.2, D14.2 (A), D15.4 (-), Q20.1 (E), R38.2
- new net 59 VAC: K2.1 (Pin_1), K2.2 (Pin_2), R59.2, R60.2
- new net GND: C10.2, C29.2, C33.1, C6.2, C7.2, C9.2, D17.2 (A), IC2.5 (B+INPUT), K1.1 (Pin_1), R2.2, R57.2, R63.1
- new net GNDPWR: C13.2, C14.1, C15.2, C16.1, C17.2, C18.1, C21.2, C22.1, C23.2, C24.1, C33.2, D7.2 (A), D8.1 (K), IC1.2 (A-INPUT), IC1.3 (A+INPUT), K3.1 (Pin_1)
- new net P_AMP_INPUT: K1.2 (Pin_2), R1.1
- new net P_AMP_OUTPUT: K3.3 (Pin_3), Q26.1 (E), Q27.1 (E), R43.1, R44.2, R45.2, R46.1, R49.2, R50.1, R55.2, R56.2, R58.2
Other:
- note added: "+"
- note added: "-"
