File: PowerAmp.kicad_sch (KiCad schematic)
At the start: 156 parts, among them IC1 NJM4580D-D, IC2 NJM4580D-D, K1 Conn_01x02_Pin, K2 Conn_01x02_Pin, K3 Conn_01x04_Pin, K4 Conn_01x03_Pin, Q1 2SA1376-K/U, Q10 2SA1145-Y, Q11 2SC2705-Y, Q12 2SC2705-Y, Q13 2SA1145-Y, Q14 2SA1145-Y, Q15 2SC2705-Y, Q16 2SC2705-Y, Q17 2SA1507-S/T, Q18 2SC3902-S/T, Q19 2SC4793, Q2 2SA1376-K/U, Q20 2SA1837, Q21 2SC5949-O, Q22 2SA2121-O, Q23 2SC5949-O, Q24 2SA2121-O, Q25 2SC3902-S/T, Q26 2SA1376-K/U, Q27 2SC3478-K/U, Q3 2SC3478-K/U, Q4 2SC3478-K/U, Q5 2SC3478-K/U, Q6 2SC3478-K/U, Q7 2SA1376-K/U, Q8 2SA1376-K/U, Q9 2SA1145-Y

Commit message: Fixes to schematic and add datasheets
Parts:
- Q17, Q18: footprint Package_TO_SOT_THT:TO-92_Inline -> Package_TO_SOT_THT:TO-126-3_Vertical
- Q25: value 2SC3902-S/T -> 2SC4685
Connections:
- net -78.9V: now also Q20.3 (E); no longer Q20.1 (E)
- net at R41.1, R45.1, R51.1: now also Q21.3 (E); no longer Q21.1 (E)
- net at Q24.1 (B): now also Q22.1 (B), R40.1; no longer R50.2
- net at C10.1, D4.1 (K), D6.1 (K)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: now also Q20.1 (B); no longer Q20.3 (B)
- net at R36.2, R39.1: now also Q19.3 (E); no longer Q19.1 (E)
- net at R42.2, R46.2, R52.1: now also Q22.3 (E); no longer Q22.1 (E)
- net at Q23.1 (B): now also Q21.1 (B), R39.2; no longer R49.1
- net at C9.1, D3.2 (A), D5.2 (A)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: now also Q19.1 (B); no longer Q19.3 (B)
- new net: Q24.3 (E), R50.2
- new net: Q23.3 (E), R49.1
Other:
- moved on the sheet: C33, D15, K2, K4, R59, R60, R66, R67

Commit message: Initial PCB layout
Parts:
- C1, C2, C3, C4: footprint (none) -> Capacitor_THT:C_Rect_L7.2mm_W5.5mm_P5.00mm_FKS2_FKP2_MKS2_MKP2; mfr_id (none) -> WIMA FKP2J014701I00HSSD
- C10, C9: footprint (none) -> Capacitor_THT:C_Disc_D5.0mm_W2.5mm_P5.00mm; mfr_id (none) -> KEMET C322C331JCG5TA
- C11, C12: footprint (none) -> Capacitor_THT:C_Rect_L7.2mm_W5.5mm_P5.00mm_FKS2_FKP2_MKS2_MKP2; mfr_id (none) -> WIMA FKP2D016801G00HA00
- C13, C14, C15, C16: footprint (none) -> Capacitor_THT:CP_Radial_D12.5mm_P5.00mm; mfr_id (none) -> Panasonic EEU-FS2A331L
- C17, C18, C6, C7: footprint (none) -> Capacitor_THT:C_Rect_L7.2mm_W4.5mm_P5.00mm_FKS2_FKP2_MKS2_MKP2; mfr_id (none) -> WIMA MKP2F031001F00
- C19, C20: footprint (none) -> Capacitor_THT:CP_Radial_D18.0mm_P7.50mm; mfr_id (none) -> Rubycon 50ZLJ3300M18X35.5
- C21, C22: footprint (none) -> Capacitor_THT:CP_Radial_D10.0mm_P5.00mm; mfr_id (none) -> Nichicon UCY2D220MPD
- C23, C24: footprint (none) -> Capacitor_THT:CP_Radial_D8.0mm_P3.50mm; mfr_id (none) -> Nichicon UKA1H101MPD
- C25: renamed from C33; footprint (none) -> Capacitor_THT:C_Rect_L7.2mm_W3.0mm_P5.00mm_FKS2_FKP2_MKS2_MKP2; mfr_id (none) -> WIMA MKP2G022201E00JO00
- C26: footprint (none) -> Capacitor_THT:CP_Radial_D8.0mm_P3.50mm; mfr_id (none) -> Nichicon UES1H100MPM
- C28: footprint (none) -> Capacitor_THT:CP_Radial_D8.0mm_P3.50mm; mfr_id (none) -> Nichicon UKZ2A100MPM
- C29: footprint (none) -> Capacitor_THT:C_Rect_L7.2mm_W4.5mm_P5.00mm_FKS2_FKP2_MKS2_MKP2; mfr_id (none) -> WIMA FKP2D011501D00HSSD
- C30, C31: footprint (none) -> Capacitor_THT:C_Rect_L7.2mm_W4.5mm_P5.00mm_FKS2_FKP2_MKS2_MKP2; mfr_id (none) -> WIMA FKP2D003301D00HA00
- C32: footprint (none) -> Capacitor_THT:C_Rect_L7.2mm_W3.0mm_P5.00mm_FKS2_FKP2_MKS2_MKP2; mfr_id (none) -> WIMA MKP2G022201E00JO00
- D1, D16, D17, D18, D19, D2, D20, D21, D7, D8: footprint (none) -> Diode_THT:D_A-405_P7.62mm_Horizontal; mfr_id (none) -> * CHANGE
- D10, D11, D12, D13, D14, D3, D4, D5, D6, D9: footprint Diode_THT:D_DO-35_SOD27_P7.62mm_Horizontal -> Diode_THT:D_A-405_P7.62mm_Horizontal; mfr_id (none) -> * CHANGE
- D15: footprint Diode_THT:Diode_Bridge_Vishay_GBU -> Diode_THT:Diode_Bridge_19.0x3.5x10.0mm_P5.0mm; mfr_id (none) -> * CHANGE
- IC1, IC2: footprint DIP8_NWJ -> local_amp_footprints:DIP8_NMD
- K1, K2: footprint (none) -> Connector_PinSocket_2.54mm:PinSocket_1x02_P2.54mm_Vertical; mfr_id (none) -> * CHANGE
- K3: footprint (none) -> Connector_PinSocket_2.54mm:PinSocket_1x04_P2.54mm_Vertical; mfr_id (none) -> * CHANGE
- K4: footprint (none) -> Connector_PinSocket_2.54mm:PinSocket_1x03_P2.54mm_Vertical; mfr_id (none) -> * CHANGE
- Q17, Q18: footprint Package_TO_SOT_THT:TO-126-3_Vertical -> local_amp_footprints:TO-126_TOS
- Q19, Q20: footprint Package_TO_SOT_THT:TO-92_Inline -> local_amp_footprints:TO-220_2-10R1A_TOS
- Q21, Q22, Q23, Q24: footprint Package_TO_SOT_THT:TO-92_Inline -> local_amp_footprints:TO-3PL_TOS
- Q25: footprint Package_TO_SOT_THT:TO-92_Inline -> local_amp_footprints:TO-126_TOS
- R1: footprint (none) -> Resistor_THT:R_Axial_DIN0207_L6.3mm_D2.5mm_P10.16mm_Horizontal; mfr_id (none) -> YAGEO MF0207FRE52-470R
- R10, R11, R12, R17, R18, R19, R20, R9: footprint (none) -> Resistor_THT:R_Axial_DIN0207_L6.3mm_D2.5mm_P10.16mm_Horizontal; mfr_id (none) -> YAGEO MF0207FTE52-22R
- R13, R14, R15, R16: footprint (none) -> Resistor_THT:R_Axial_DIN0207_L6.3mm_D2.5mm_P10.16mm_Horizontal; mfr_id (none) -> YAGEO MF0207FTE52-2K4
- R2: footprint (none) -> Resistor_THT:R_Axial_DIN0207_L6.3mm_D2.5mm_P10.16mm_Horizontal; mfr_id (none) -> YAGEO MF0207FTE52-24K
- R21, R22, R23, R24: footprint (none) -> Resistor_THT:R_Axial_DIN0207_L6.3mm_D2.5mm_P10.16mm_Horizontal; mfr_id (none) -> YAGEO MF0207FTE52-5K6
- R25, R26, R27, R28, R33: footprint (none) -> Resistor_THT:R_Axial_DIN0207_L6.3mm_D2.5mm_P10.16mm_Horizontal; mfr_id (none) -> YAGEO MF0207FTE52-1K
- R29, R30, R31, R32: footprint (none) -> Resistor_THT:R_Axial_DIN0207_L6.3mm_D2.5mm_P10.16mm_Horizontal; mfr_id (none) -> Vishay NFR25H0001500JR500
- R3, R4: footprint (none) -> Resistor_THT:R_Axial_DIN0207_L6.3mm_D2.5mm_P10.16mm_Horizontal; mfr_id (none) -> YAGEO MF0207FTE52-100R
- R34: footprint (none) -> Resistor_THT:R_Axial_DIN0207_L6.3mm_D2.5mm_P10.16mm_Horizontal; mfr_id (none) -> YAGEO MF0207FTE52-240R
- R35: footprint (none) -> Resistor_THT:R_Axial_DIN0207_L6.3mm_D2.5mm_P10.16mm_Horizontal; mfr_id (none) -> YAGEO MF0207FTE52-75K
- R36: footprint (none) -> Resistor_THT:R_Axial_DIN0414_L11.9mm_D4.5mm_P15.24mm_Horizontal; mfr_id (none) -> KOA MOS2CT52A470J
- R37, R38, R66, R67: footprint (none) -> Resistor_THT:R_Axial_DIN0414_L11.9mm_D4.5mm_P15.24mm_Horizontal; mfr_id (none) -> KOA MOS2CT52R1000F
- R39, R40: footprint (none) -> Resistor_THT:R_Axial_DIN0207_L6.3mm_D2.5mm_P10.16mm_Horizontal; mfr_id (none) -> YAGEO MF0207FRE52-2R2
- R41, R42: footprint (none) -> Resistor_THT:R_Axial_DIN0207_L6.3mm_D2.5mm_P10.16mm_Horizontal; mfr_id (none) -> YAGEO MF0207FTE52-680R
- R43, R44: footprint (none) -> Resistor_THT:R_Axial_DIN0207_L6.3mm_D2.5mm_P10.16mm_Horizontal; mfr_id (none) -> YAGEO MF0207FRE52-390R
- R45, R46, R49, R50: footprint (none) -> Resistor_THT:R_Box_L14.0mm_W5.0mm_P9.00mm; mfr_id (none) -> KOA BPR58CR22J
- R5, R6, R7, R8: footprint (none) -> Resistor_THT:R_Axial_DIN0207_L6.3mm_D2.5mm_P10.16mm_Horizontal; mfr_id (none) -> YAGEO MF0207FTE52-15K
- R51, R52: footprint (none) -> Resistor_THT:R_Axial_DIN0207_L6.3mm_D2.5mm_P10.16mm_Horizontal; mfr_id (none) -> YAGEO MF0207FRE52-330R
- R53, R54, R71, R72: footprint (none) -> Resistor_THT:R_Axial_DIN0617_L17.0mm_D6.0mm_P20.32mm_Horizontal; mfr_id (none) -> KOA MOS3CT631R562J
- R55, R56: footprint (none) -> Resistor_THT:R_Axial_DIN0411_L9.9mm_D3.6mm_P15.24mm_Horizontal; mfr_id (none) -> Vishay Dale CMF504K4200FHEB
- R57, R58: footprint (none) -> Resistor_THT:R_Axial_DIN0207_L6.3mm_D2.5mm_P10.16mm_Horizontal; mfr_id (none) -> YAGEO MF0207FTE52-33K
- R59, R60: footprint (none) -> Resistor_THT:R_Axial_DIN0207_L6.3mm_D2.5mm_P10.16mm_Horizontal; mfr_id (none) -> TE Connectivity FRN25JR47
- R61: footprint (none) -> Resistor_THT:R_Axial_DIN0617_L17.0mm_D6.0mm_P20.32mm_Horizontal; mfr_id (none) -> Vishay PR03000202211FAC00
- R62, R64: footprint (none) -> Resistor_THT:R_Axial_DIN0411_L9.9mm_D3.6mm_P15.24mm_Horizontal; mfr_id (none) -> Vishay Dale CMF50332R00FHEB
- R63: footprint (none) -> Resistor_THT:R_Axial_DIN0207_L6.3mm_D2.5mm_P10.16mm_Horizontal; mfr_id (none) -> YAGEO MF0207FTE52-270K
- R68, R69: footprint (none) -> Resistor_THT:R_Axial_DIN0204_L3.6mm_D1.6mm_P7.62mm_Horizontal; mfr_id (none) -> Vishay Dale CMF501K0000FHEA
- R70: footprint (none) -> Resistor_THT:R_Axial_DIN0204_L3.6mm_D1.6mm_P7.62mm_Horizontal; mfr_id (none) -> Vishay Dale CMF50715R00FHEB
- TP1: footprint (none) -> Connector_PinHeader_2.54mm:PinHeader_1x02_P2.54mm_Vertical
- TPA_1V2, TPB_1V2: footprint (none) -> Connector_PinHeader_2.54mm:PinHeader_1x01_P2.54mm_Vertical
- VR1: footprint (none) -> Potentiometer_THT:Potentiometer_ACP_CA6-H2,5_Horizontal; mfr_id (none) -> * CHANGE

Commit message: PCB layout
Parts:
- IC1, IC2: footprint local_amp_footprints:DIP8_NMD -> Package_DIP:DIP-8_W7.62mm
- Q17, Q18, Q25: footprint local_amp_footprints:TO-126_TOS -> Package_TO_SOT_THT:TO-126-3_Vertical
- Q19, Q20: footprint local_amp_footprints:TO-220_2-10R1A_TOS -> Package_TO_SOT_THT:TO-220-3_Vertical
- Q21, Q22, Q23, Q24: footprint local_amp_footprints:TO-3PL_TOS -> Package_TO_SOT_THT:TO-3P-3_Vertical
Changed lines of the file:
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@@
 			)
 		)
-		(property "Footprint" "local_amp_footprints:TO-3PL_TOS"
+		(property "Footprint" "Package_TO_SOT_THT:TO-3P-3_Vertical"
 			(at 469.9 212.725 0)
 			(hide yes)
@@
 			)
 		)
-		(property "Footprint" "local_amp_footprints:DIP8_NMD"
+		(property "Footprint" "Package_DIP:DIP-8_W7.62mm"
 			(at 65.532 162.052 0)
 			(hide yes)
@@
 			)
 		)
-		(property "Footprint" "local_amp_footprints:TO-126_TOS"
+		(property "Footprint" "Package_TO_SOT_THT:TO-126-3_Vertical"
 			(at 351.79 133.985 0)
 			(hide yes)
@@
 			)
 		)
-		(property "Footprint" "local_amp_footprints:TO-220_2-10R1A_TOS"
+		(property "Footprint" "Package_TO_SOT_THT:TO-220-3_Vertical"
 			(at 405.13 150.495 0)
 			(hide yes)
@@
 			)
 		)
-		(property "Footprint" "local_amp_footprints:TO-3PL_TOS"
+		(property "Footprint" "Package_TO_SOT_THT:TO-3P-3_Vertical"
 			(at 447.04 212.725 0)
 			(hide yes)
@@
 			)
 		)
-		(property "Footprint" "local_amp_footprints:TO-3PL_TOS"
+		(property "Footprint" "Package_TO_SOT_THT:TO-3P-3_Vertical"
 			(at 469.9 150.495 0)
 			(hide yes)
@@
 			)
 		)
-		(property "Footprint" "local_amp_footprints:TO-126_TOS"
+		(property "Footprint" "Package_TO_SOT_THT:TO-126-3_Vertical"
 			(at 351.79 229.235 0)
 			(hide yes)
@@
 			)
 		)
-		(property "Footprint" "local_amp_footprints:TO-220_2-10R1A_TOS"
+		(property "Footprint" "Package_TO_SOT_THT:TO-220-3_Vertical"
 			(at 405.13 216.535 0)
 			(hide yes)
@@
 			)
 		)
-		(property "Footprint" "local_amp_footprints:TO-126_TOS"
+		(property "Footprint" "Package_TO_SOT_THT:TO-126-3_Vertical"
 			(at 351.79 183.515 0)
 			(hide yes)
@@
 			)
 		)
-		(property "Footprint" "local_amp_footprints:DIP8_NMD"
+		(property "Footprint" "Package_DIP:DIP-8_W7.62mm"
 			(at 74.168 282.702 0)
 			(hide yes)
@@
 			)
 		)
-		(property "Footprint" "local_amp_footprints:TO-3PL_TOS"
+		(property "Footprint" "Package_TO_SOT_THT:TO-3P-3_Vertical"
 			(at 447.04 150.495 0)
 			(hide yes)

Commit message: PCB layout
Connections:
- net 59 VAC: no longer names the net of K2.1 (Pin_1), R59.2
- net 59 VAC: no longer K2.2 (Pin_2), R60.2
- new net: K2.2 (Pin_2), R60.2
Changed lines of the file:
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@@
 	)
 	(junction
-		(at 300.99 374.65)
-		(diameter 0)
-		(color 0 0 0 0)
-	)
-	(junction
 		(at 501.65 227.33)
 		(diameter 0)
@@
 	)
 	(junction
-		(at 313.69 372.11)
-		(diameter 0)
-		(color 0 0 0 0)
-	)
-	(junction
 		(at 501.65 189.23)
 		(diameter 0)
@@
 	(wire
 		(pts
-			(xy 313.69 363.22) (xy 313.69 372.11)
-		)
-		(stroke
-			(width 0)
-			(type default)
-		)
-	)
-	(wire
-		(pts
 			(xy 278.13 281.94) (xy 278.13 284.48)
 		)
@@
 	(wire
 		(pts
-			(xy 289.56 372.11) (xy 313.69 372.11)
+			(xy 289.56 372.11) (xy 325.12 372.11)
 		)
 		(stroke
@@
 	(wire
 		(pts
-			(xy 313.69 372.11) (xy 325.12 372.11)
-		)
-		(stroke
-			(width 0)
-			(type default)
-		)
-	)
-	(wire
-		(pts
 			(xy 34.29 252.73) (xy 34.29 265.43)
 		)
@@
 	(wire
 		(pts
-			(xy 300.99 363.22) (xy 300.99 374.65)
-		)
-		(stroke
-			(width 0)
-			(type default)
-		)
-	)
-	(wire
-		(pts
 			(xy 161.29 287.02) (xy 161.29 314.96)
 		)
@@
 	)
 	(symbol
-		(lib_id "power:VAC")
-		(at 300.99 363.22 0)
-		(unit 1)
-		(body_style 1)
-		(exclude_from_sim no)
-		(in_bom yes)
-		(on_board yes)
-		(in_pos_files yes)
-		(dnp no)
-		(fields_autoplaced yes)
-		(property "Reference" "#PWR037"
-			(at 300.99 365.76 0)
-			(hide yes)
-			(show_name no)
-			(do_not_autoplace no)
-			(effects
-				(font
-					(size 1.27 1.27)
-				)
-			)
-		)
-		(property "Value" "59 VAC"
-			(at 300.99 355.6 0)
-			(show_name no)
-			(do_not_autoplace no)
-			(effects
-				(font
-					(size 1.27 1.27)
-				)
-			)
-		)
-		(property "Footprint" ""
-			(at 300.99 363.22 0)
-			(hide yes)
-			(show_name no)
-			(do_not_autoplace no)
-			(effects
-				(font
-					(size 1.27 1.27)
-				)
-			)
-		)
-		(property "Datasheet" ""
-			(at 300.99 363.22 0)
-			(hide yes)
-			(show_name no)
-			(do_not_autoplace no)
-			(effects
-				(font
-					(size 1.27 1.27)
-				)
-			)
-		)
-		(property "Description" "Power symbol creates a global label with name \"VAC\""
-			(at 300.99 363.22 0)
-			(hide yes)
-			(show_name no)
-			(do_not_autoplace no)
-			(effects
-				(font
-					(size 1.27 1.27)
-				)
-			)
-		)
-		(pin "1"
-		)
-		(instances
-			(project "PowerAmp"
-				(path "/f3a40bfa-83f5-46f5-84c7-bcd44139818c"
-					(reference "#PWR037")
-					(unit 1)
-				)
-			)
-		)
-	)
-	(symbol
 		(lib_name "2SA1015_3")
 		(lib_id "Transistor_BJT:2SA1015")
@@
 					(unit 1)
 				)
-			)
-		)
-	)
-	(symbol
-		(lib_id "power:VAC")
-		(at 313.69 363.22 0)
-		(unit 1)
-		(body_style 1)
-		(exclude_from_sim no)
-		(in_bom yes)
-		(on_board yes)
-		(in_pos_files yes)
-		(dnp no)
-		(fields_autoplaced yes)
-		(property "Reference" "#PWR038"
-			(at 313.69 365.76 0)
-			(hide yes)
-			(show_name no)
-			(do_not_autoplace no)
-			(effects
-				(font
-					(size 1.27 1.27)
-				)
-			)
-		)
-		(property "Value" "59 VAC"
-			(at 313.69 355.6 0)
-			(show_name no)
-			(do_not_autoplace no)
-			(effects
-				(font
-					(size 1.27 1.27)
-				)
-			)
-		)
-		(property "Footprint" ""
-			(at 313.69 363.22 0)
-			(hide yes)
-			(show_name no)
-			(do_not_autoplace no)
-			(effects
-				(font
-					(size 1.27 1.27)
-				)
-			)
-		)
-		(property "Datasheet" ""
-			(at 313.69 363.22 0)
-			(hide yes)
-			(show_name no)
-			(do_not_autoplace no)
-			(effects
-				(font
-					(size 1.27 1.27)
-				)
-			)
-		)
-		(property "Description" "Power symbol creates a global label with name \"VAC\""
-			(at 313.69 363.22 0)
-			(hide yes)
-			(show_name no)
-			(do_not_autoplace no)
-			(effects
-				(font
-					(size 1.27 1.27)
-				)
-			)
-		)
-		(pin "1"
-		)
-		(instances
-			(project "PowerAmp"
-				(path "/f3a40bfa-83f5-46f5-84c7-bcd44139818c"
-					(reference "#PWR038")
-					(unit 1)
-				)
