File: PowerAmp.kicad_pcb (KiCad board)
At the start: 2 copper layers, 156 parts, among them IC1 NJM4580D-D, IC2 NJM4580D-D, K1 Conn_01x02_Pin, K2 Conn_01x02_Pin, K3 Conn_01x04_Pin, K4 Conn_01x03_Pin, Q1 2SA1376-K/U, Q10 2SA1145-Y, Q11 2SC2705-Y, Q12 2SC2705-Y, Q13 2SA1145-Y, Q14 2SA1145-Y, Q15 2SC2705-Y, Q16 2SC2705-Y, Q17 2SA1507-S/T, Q18 2SC3902-S/T, Q19 2SC4793, Q2 2SA1376-K/U, Q20 2SA1837, Q21 2SC5949-O, Q22 2SA2121-O, Q23 2SC5949-O, Q24 2SA2121-O, Q25 2SC4685, Q26 2SA1376-K/U, Q27 2SC3478-K/U, Q3 2SC3478-K/U, Q4 2SC3478-K/U, Q5 2SC3478-K/U, Q6 2SC3478-K/U, Q7 2SA1376-K/U, Q8 2SA1376-K/U, Q9 2SA1145-Y

Commit message: PCB layout
Parts:
- IC1, IC2: footprint local_amp_footprints:DIP8_NMD -> Package_DIP:DIP-8_W7.62mm
- Q17, Q18, Q25: footprint local_amp_footprints:TO-126_TOS -> Package_TO_SOT_THT:TO-126-3_Vertical
- Q19, Q20: footprint local_amp_footprints:TO-220_2-10R1A_TOS -> Package_TO_SOT_THT:TO-220-3_Vertical
- Q21, Q22, Q23, Q24: footprint local_amp_footprints:TO-3PL_TOS -> Package_TO_SOT_THT:TO-3P-3_Vertical
- R61: footprint Resistor_THT:R_Axial_DIN0617_L17.0mm_D6.0mm_P20.32mm_Horizontal -> Resistor_THT:R_Axial_DIN0411_L9.9mm_D3.6mm_P15.24mm_Horizontal
- moved C10 442.5 mm to (-99.9, 236.8), turned to 90 degrees
- moved R40 417.7 mm to (-76.2, 231.7), turned to -90 degrees
- moved C22 394.7 mm to (-70.7, 197.9), turned to 90 degrees
- moved D4 384.1 mm to (-94.8, 230.4), turned to -90 degrees
- moved D6 375.4 mm to (-91.0, 230.4), turned to -90 degrees
- moved C18 373.0 mm to (-73.2, 184.2)
- moved R42 368.2 mm to (-47.6, 199.4), turned to -90 degrees
- moved D14 364.6 mm to (-80.8, 218.4), turned to -90 degrees
- moved R44 364.0 mm to (-51.5, 199.4), turned to -90 degrees
- moved TP1 360.7 mm to (-62.5, 153.7), turned to 90 degrees
- moved C25 357.3 mm to (-17.1, 216.5), turned to -90 degrees
- moved C30 352.0 mm to (-33.7, 202.5), turned to 90 degrees
- moved R35 351.7 mm to (-41.3, 225.4)
- moved C2 347.7 mm to (-25.4, 173.9), turned to 90 degrees
- moved C4 343.9 mm to (-41.9, 168.9), turned to -90 degrees
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
Commit message: PCB routing
Parts:
- moved R62 19.1 mm to (-5.08, 191.8), turned to 90 degrees
- moved R15 10.2 mm to (20.3, 166.4), turned to -90 degrees
- moved C3 5.04 mm to (25.4, 173.9), turned to 90 degrees
- moved D15 3.81 mm to (8.87, 196.4)
- moved R55 3.81 mm to (3.81, 176.5)
- moved R56 3.81 mm to (-0.64, 176.5)
- moved R61 3.81 mm to (8.89, 176.5)
- moved R64 3.81 mm to (-9.53, 176.5)
- moved C29 1.67 mm to (-8.26, 161.2)
- moved R2 1.21 mm to (-3.81, 163.5)
- moved R1 0.64 mm to (2.54, 156.6)
- moved R63 0.64 mm to (-0.64, 156.6)
Routing:
- net Net-(R17-Pad1): track 0.00 -> 89.6 mm
- net Net-(R3-Pad1): track 0.00 -> 85.3 mm
- net Net-(D20-K): track 0.00 -> 6.15 mm
- net Net-(C2-Pad1): track 0.00 -> 6.13 mm
- added copper zone on F.Cu, net GND

Commit message: PCB layout
Parts:
- R61: footprint Resistor_THT:R_Axial_DIN0411_L9.9mm_D3.6mm_P15.24mm_Horizontal -> Resistor_THT:R_Axial_DIN0617_L17.0mm_D6.0mm_P20.32mm_Horizontal
- moved C7 67.5 mm to (33.7, 187.3), turned to 90 degrees
- moved C6 67.5 mm to (-33.7, 187.3), turned to 90 degrees
- moved R53 20.3 mm to (88.8, 174.0), turned to 90 degrees
- moved R71 20.3 mm to (99.0, 174.0), turned to 90 degrees
- moved R45 17.9 mm to (9.53, 247.0), turned to 90 degrees
- moved R49 17.9 mm to (41.9, 247.0), turned to 90 degrees
- moved R39 17.3 mm to (82.5, 236.9)
- moved R37 17.1 mm to (57.8, 208.9), turned to 90 degrees
- moved R38 13.3 mm to (-58.4, 193.7), turned to -90 degrees
- moved R50 12.1 mm to (-32.4, 238.0)
- moved R46 11.3 mm to (-64.8, 238.0)
- moved R33 10.6 mm to (64.8, 163.8), turned to 90 degrees
- moved R51 10.5 mm to (-61.6, 168.3), turned to 90 degrees
- moved R60 10.5 mm to (-3.00, 196.5), turned to -90 degrees
- moved R59 10.5 mm to (-6.35, 196.5), turned to -90 degrees
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Connections:
- K2 pad 1: 59 VAC -> Net-(K2-Pin_1)
- K2 pad 2: 59 VAC -> Net-(K2-Pin_2)
- R59 pad 2: 59 VAC -> Net-(K2-Pin_1)
- R60 pad 2: 59 VAC -> Net-(K2-Pin_2)
Routing:
- net Net-(D7-K): track 0.00 -> 284.5 mm, vias 0 -> 5
- net Net-(Q21-E): track 0.00 -> 189.8 mm
- net Net-(D4-K): track 0.00 -> 151.3 mm, vias 0 -> 1
- net Net-(D2-K): track 0.00 -> 131.1 mm, vias 0 -> 1
- net Net-(Q22-E): track 0.00 -> 119.3 mm
- net 78.9V_negative: track 0.00 -> 104.4 mm, vias 0 -> 2
- net Net-(Q11-C): track 0.00 -> 103.2 mm, vias 0 -> 2
- net 74.8V_negative: track 0.00 -> 102.6 mm, vias 0 -> 1
- net Net-(D1-A): track 0.00 -> 90.8 mm, vias 0 -> 1
- net Net-(R17-Pad1): track 89.6 -> 0.00 mm
- net Net-(R3-Pad1): track 85.3 -> 0.00 mm
- net Net-(Q10-C): track 0.00 -> 77.1 mm
- net Net-(Q22-B): track 0.00 -> 77.0 mm, vias 0 -> 1
- net Net-(D8-A): track 0.00 -> 59.5 mm
- net Net-(D4-A): track 0.00 -> 54.5 mm
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- added copper zone on F.Cu, net +66V
- added copper zone on F.Cu, net -66V
- added copper zone on B.Cu, net 78.9V_negative
- added copper zone on B.Cu, net 78.9V_positive
- added copper zone on F.Cu, net Net-(D7-K)
- added copper zone on F.Cu, net Net-(D8-A)
